Commit message: khan_msgs and khan_description compiling w amnet

File: khan_description/urdf/khan.gazebo.xacro (robot description, xacro)
@@ -24,4 +24,5 @@
   <xacro:include filename="$(find khan_description)/urdf/khan.urdf.xacro" />
   <!-- Gazebo plugin for ROS Control -->
+  <!-- TODO: Determine if this is necessary for ROS2 -->
   <gazebo>
     <plugin name="gazebo_ros_control" filename="libgazebo_ros_control.so">

File: khan_description/urdf/khan.urdf.xacro (robot description, xacro)
@@ -25,10 +25,10 @@
   <xacro:include filename="$(find khan_description)/urdf/decorations.urdf.xacro" />
   <xacro:include filename="$(find khan_description)/urdf/wheel.urdf.xacro" />
-  <property name="M_PI" value="3.14159"/>
+  <xacro:property name="M_PI" value="3.14159"/>
   <!-- Base Size -->
-  <property name="base_x_size" value="0.245" />
-  <property name="base_y_size" value="0.153" />
-  <property name="base_z_size" value="0.074" />
-  <property name="base_z_clearance" value="0.021" />
+  <xacro:property name="base_x_size" value="0.245" />
+  <xacro:property name="base_y_size" value="0.153" />
+  <xacro:property name="base_z_size" value="0.074" />
+  <xacro:property name="base_z_clearance" value="0.021" />
   <!-- Wheel Mounting Positions -->
   <xacro:property name="wheelbase" value="0.185" />
